File: esp-wroom-32-break.sch (KiCad schematic (older format))
At the start: 7 parts

Commit message: Update schema with using 18 pins connectors etc
Parts:
- removed CON?: SD_Card, 10067847-001, symbol SD_Card
- removed D? (x2): LED, symbol LED
- removed U?: FT232RL, SSOP-28, symbol FT232RL
- added C?: 0.1uf, symbol C
- added CON?: Micro_SD_Card, symbol Micro_SD_Card
- added IC?: FT232RQ, ftdi4-QFN-32, symbol FT232RQ
- added P? (x2): CONN_01X18, symbol CONN_01X18
- added P?: Switch, symbol CONN_01X02
- added R?: 10K, symbol R
- P?: symbol USB_OTG -> USB_OTG-RESCUE-esp-wroom-32-break
Connections:
- net labels added: IO12, IO13, IO14, IO15, IO16, IO17, IO18, IO19, IO2, IO21, IO22, IO23, IO25, IO26, IO27, IO32, IO33, IO34, IO35, IO4, IO5, SVN, SVP, VCC
- net labels removed: CTS, DTR
- wire segments 27 -> 37
- no-connect marks 14 -> 23

Commit message: Assign component footprints and generated net file
Parts:
- removed U?: AMS1117, SOT-223, symbol LT1129IST-3.3
- added C2, C4: 0.1uf, Capacitors_SMD:C_0603, symbol C
- added C3, C5: 10uf, Capacitors_SMD:C_0603, symbol C
- added D1: D, Diodes_SMD:D_0805, symbol D
- added U2: NJU7223DL1-33, TO_SOT_Packages_SMD:TO-252-2Lead, symbol NJU7223DL1-33
- C1: renamed from C?; footprint (none) -> Capacitors_SMD:C_0603
- CON1: renamed from CON?; footprint (none) -> Connectors_Hirose:microSD_Card_Receptacle_Hirose_DM3AT-SF-PEJM5
- IC1: renamed from IC?; footprint ftdi4-QFN-32 -> ftdi4:ftdi4-QFN-32
- P1, P2: renamed from P?; footprint (none) -> Pin_Headers:Pin_Header_Straight_1x18_Pitch2.54mm
- P3: renamed from P?; footprint (none) -> usb_micro_b:USB_MICRO_B-HIROSE-ZX62R-B-5P
- P4: renamed from P?; footprint (none) -> Buttons_Switches_SMD:SW_SPST_B3S-1000
- R1: renamed from R?; footprint (none) -> Resistors_SMD:R_0603
- gave numbers to parts that had none: 1
Connections:
- net +3V3: now also C2.1, C3.1, U2.1 (Vout)
- net +5V: now also D1.2 (A)
- net GND: now also P3.6 (shield), C2.2, C3.2, C4.2, C5.2, U2.3 (GND)
- net VCC: now also C4.1, C5.1, D1.1 (K), U2.2 (Vin)
