File: _saved_esp-wroom-32-break.sch (KiCad schematic (older format))
At the start: 17 parts, among them CON1 Micro_SD_Card, IC1 FT232RQ, P1 CONN_01X18, P2 CONN_01X18, P3 USB_OTG, P4 Switch, U1 ESP32-WROOM, U2 NJU7223DL1-33

Commit message: Put footprints
Parts:
- gave numbers to parts that had none: 2
Changed lines of the file:
@@
 RXDtoTXD0
 $Comp
-L +3.3V #PWR06
+L +3.3V #PWR05
 U 1 1 586B9054
 P 4300 3150
-F 0 "#PWR06" H 4300 3000 50  0001 C CNN
+F 0 "#PWR05" H 4300 3000 50  0001 C CNN
 F 1 "+3.3V" H 4300 3290 50  0000 C CNN
 F 2 "" H 4300 3150 50  0000 C CNN
@@
 $EndComp
 $Comp
-L +3.3V #PWR07
+L +3.3V #PWR06
 U 1 1 586B907B
 P 7850 5800
-F 0 "#PWR07" H 7850 5650 50  0001 C CNN
+F 0 "#PWR06" H 7850 5650 50  0001 C CNN
 F 1 "+3.3V" H 7850 5940 50  0000 C CNN
 F 2 "" H 7850 5800 50  0000 C CNN
@@
 $EndComp
 $Comp
-L GND #PWR08
+L GND #PWR07
 U 1 1 586B90BE
 P 7850 6000
-F 0 "#PWR08" H 7850 5750 50  0001 C CNN
+F 0 "#PWR07" H 7850 5750 50  0001 C CNN
 F 1 "GND" H 7850 5850 50  0000 C CNN
 F 2 "" H 7850 6000 50  0000 C CNN
@@
 $EndComp
 $Comp
-L +3.3V #PWR09
+L +3.3V #PWR08
 U 1 1 586B92DC
 P 3950 6250
-F 0 "#PWR09" H 3950 6100 50  0001 C CNN
+F 0 "#PWR08" H 3950 6100 50  0001 C CNN
 F 1 "+3.3V" H 3950 6390 50  0000 C CNN
 F 2 "" H 3950 6250 50  0000 C CNN
@@
 $EndComp
 $Comp
-L GND #PWR010
+L GND #PWR09
 U 1 1 586B9430
 P 3950 6450
-F 0 "#PWR010" H 3950 6200 50  0001 C CNN
+F 0 "#PWR09" H 3950 6200 50  0001 C CNN
 F 1 "GND" H 3950 6300 50  0000 C CNN
 F 2 "" H 3950 6450 50  0000 C CNN
@@
 $EndComp
 $Comp
-L GND #PWR011
+L GND #PWR010
 U 1 1 58946005
 P 6100 6850
-F 0 "#PWR011" H 6100 6600 50  0001 C CNN
+F 0 "#PWR010" H 6100 6600 50  0001 C CNN
 F 1 "GND" H 6100 6700 50  0000 C CNN
 F 2 "" H 6100 6850 50  0000 C CNN
@@
 $EndComp
 $Comp
-L +3.3V #PWR012
+L +3.3V #PWR011
 U 1 1 58948A12
 P 1200 3050
-F 0 "#PWR012" H 1200 2900 50  0001 C CNN
+F 0 "#PWR011" H 1200 2900 50  0001 C CNN
 F 1 "+3.3V" H 1200 3190 50  0000 C CNN
 F 2 "" H 1200 3050 50  0000 C CNN
@@
 $EndComp
 $Comp
-L GND #PWR013
+L GND #PWR012
 U 1 1 58948B03
 P 1350 2600
-F 0 "#PWR013" H 1350 2350 50  0001 C CNN
+F 0 "#PWR012" H 1350 2350 50  0001 C CNN
 F 1 "GND" H 1350 2450 50  0000 C CNN
 F 2 "" H 1350 2600 50  0000 C CNN
@@
 $EndComp
 $Comp
-L +3.3V #PWR014
+L +3.3V #PWR013
 U 1 1 58948C61
 P 2750 3050
-F 0 "#PWR014" H 2750 2900 50  0001 C CNN
+F 0 "#PWR013" H 2750 2900 50  0001 C CNN
 F 1 "+3.3V" H 2750 3190 50  0000 C CNN
 F 2 "" H 2750 3050 50  0000 C CNN
@@
 $EndComp
 $Comp
-L GND #PWR015
+L GND #PWR014
 U 1 1 58948C68
 P 2900 2600
-F 0 "#PWR015" H 2900 2350 50  0001 C CNN
+F 0 "#PWR014" H 2900 2350 50  0001 C CNN
 F 1 "GND" H 2900 2450 50  0000 C CNN
 F 2 "" H 2900 2600 50  0000 C CNN
@@
 $EndComp
 $Comp
-L VCC #PWR016
+L VCC #PWR015
 U 1 1 58948CFD
 P 2900 4650
-F 0 "#PWR016" H 2900 4500 50  0001 C CNN
+F 0 "#PWR015" H 2900 4500 50  0001 C CNN
 F 1 "VCC" H 2900 4800 50  0000 C CNN
 F 2 "" H 2900 4650 50  0000 C CNN
@@
 $EndComp
 $Comp
-L +3.3V #PWR017
+L +3.3V #PWR016
 U 1 1 58948D8F
 P 2900 4450
-F 0 "#PWR017" H 2900 4300 50  0001 C CNN
+F 0 "#PWR016" H 2900 4300 50  0001 C CNN
 F 1 "+3.3V" H 2900 4590 50  0000 C CNN
 F 2 "" H 2900 4450 50  0000 C CNN
@@
 $EndComp
 $Comp
-L +3.3V #PWR018
+L +3.3V #PWR017
 U 1 1 58948E57
 P 1500 4650
-F 0 "#PWR018" H 1500 4500 50  0001 C CNN
+F 0 "#PWR017" H 1500 4500 50  0001 C CNN
 F 1 "+3.3V" H 1500 4790 50  0000 C CNN
 F 2 "" H 1500 4650 50  0000 C CNN
@@
 $EndComp
 $Comp
-L GND #PWR019
+L GND #PWR018
 U 1 1 58948EC3
 P 1350 4450
-F 0 "#PWR019" H 1350 4200 50  0001 C CNN
+F 0 "#PWR018" H 1350 4200 50  0001 C CNN
 F 1 "GND" H 1350 4300 50  0000 C CNN
 F 2 "" H 1350 4450 50  0000 C CNN
@@
 $EndComp
 $Comp
-L GND #PWR020
+L GND #PWR019
 U 1 1 58948FCD
 P 2750 4250
-F 0 "#PWR020" H 2750 4000 50  0001 C CNN
+F 0 "#PWR019" H 2750 4000 50  0001 C CNN
 F 1 "GND" H 2750 4100 50  0000 C CNN
 F 2 "" H 2750 4250 50  0000 C CNN
@@
 $EndComp
 $Comp
-L +3.3V #PWR021
+L +3.3V #PWR020
 U 1 1 58949386
 P 2050 5250
-F 0 "#PWR021" H 2050 5100 50  0001 C CNN
+F 0 "#PWR020" H 2050 5100 50  0001 C CNN
 F 1 "+3.3V" H 2050 5390 50  0000 C CNN
 F 2 "" H 2050 5250 50  0000 C CNN
@@
 $EndComp
 $Comp
-L GND #PWR022
+L GND #PWR021
 U 1 1 589493DB
 P 2050 5550
-F 0 "#PWR022" H 2050 5300 50  0001 C CNN
+F 0 "#PWR021" H 2050 5300 50  0001 C CNN
 F 1 "GND" H 2050 5400 50  0000 C CNN
 F 2 "" H 2050 5550 50  0000 C CNN
@@
 $EndComp
 $Comp
-L GND #PWR023
+L GND #PWR022
 U 1 1 58949C24
 P 8300 4850
-F 0 "#PWR023" H 8300 4600 50  0001 C CNN
+F 0 "#PWR022" H 8300 4600 50  0001 C CNN
 F 1 "GND" H 8300 4700 50  0000 C CNN
 F 2 "" H 8300 4850 50  0000 C CNN
@@
 $EndComp
 $Comp
-L GND #PWR024
+L GND #PWR023
 U 1 1 5894A76D
 P 8900 5850
-F 0 "#PWR024" H 8900 5600 50  0001 C CNN
+F 0 "#PWR023" H 8900 5600 50  0001 C CNN
 F 1 "GND" H 8900 5700 50  0000 C CNN
 F 2 "" H 8900 5850 50  0000 C CNN
@@
 $EndComp
 $Comp
-L VCC #PWR025
+L VCC #PWR024
 U 1 1 5894AB64
 P 3300 5350
-F 0 "#PWR025" H 3300 5200 50  0001 C CNN
+F 0 "#PWR024" H 3300 5200 50  0001 C CNN
 F 1 "VCC" H 3300 5500 50  0000 C CNN
 F 2 "" H 3300 5350 50  0000 C CNN
@@
 $EndComp
 $Comp
-L +5V #PWR026
+L +5V #PWR025
 U 1 1 5894AB9B
 P 3000 5350
-F 0 "#PWR026" H 3000 5200 50  0001 C CNN
+F 0 "#PWR025" H 3000 5200 50  0001 C CNN
 F 1 "+5V" H 3000 5490 50  0000 C CNN
 F 2 "" H 3000 5350 50  0000 C CNN
@@
 $EndComp
 $Comp
-L +3.3V #PWR027
+L +3.3V #PWR026
 U 1 1 5894AD31
 P 9450 5550
-F 0 "#PWR027" H 9450 5400 50  0001 C CNN
+F 0 "#PWR026" H 9450 5400 50  0001 C CNN
 F 1 "+3.3V" H 9450 5690 50  0000 C CNN
 F 2 "" H 9450 5550 50  0000 C CNN
@@
 $EndComp
 $Comp
-L VCC #PWR028
+L VCC #PWR027
 U 1 1 5894ADEC
 P 10500 5550
-F 0 "#PWR028" H 10500 5400 50  0001 C CNN
+F 0 "#PWR027" H 10500 5400 50  0001 C CNN
 F 1 "VCC" H 10500 5700 50  0000 C CNN
 F 2 "" H 10500 5550 50  0000 C CNN
@@
 $EndComp
 $Comp
-L GND #PWR029
+L GND #PWR028
 U 1 1 5894B29F
 P 10800 6100
-F 0 "#PWR029" H 10800 5850 50  0001 C CNN
+F 0 "#PWR028" H 10800 5850 50  0001 C CNN
 F 1 "GND" H 10800 5950 50  0000 C CNN
 F 2 "" H 10800 6100 50  0000 C CNN
@@
 $EndComp
 $Comp
-L VCC #PWR030
+L VCC #PWR029
 U 1 1 5894BA7B
 P 6850 5800
-F 0 "#PWR030" H 6850 5650 50  0001 C CNN
+F 0 "#PWR029" H 6850 5650 50  0001 C CNN
 F 1 "VCC" H 6850 5950 50  0000 C CNN
 F 2 "" H 6850 5800 50  0000 C CNN
@@
 $EndComp
 $Comp
-L +3.3V #PWR?
+L +3.3V #PWR030
 U 1 1 5898771E
 P 7400 2700
-F 0 "#PWR?" H 7400 2550 50  0001 C CNN
+F 0 "#PWR030" H 7400 2550 50  0001 C CNN
 F 1 "+3.3V" H 7400 2840 50  0000 C CNN
 F 2 "" H 7400 2700 50  0000 C CNN
@@
 $EndComp
 $Comp
-L C C?
+L C C6
 U 1 1 589879F3
 P 7500 4750
-F 0 "C?" H 7525 4850 50  0000 L CNN
+F 0 "C6" H 7525 4850 50  0000 L CNN
 F 1 "0.1uf" H 7525 4650 50  0000 L CNN
 F 2 "Capacitors_SMD:C_0603" H 7538 4600 50  0001 C CNN
@@
 $EndComp
 $Comp
-L GND #PWR?
+L GND #PWR031
 U 1 1 58987AAB
 P 7500 4900
-F 0 "#PWR?" H 7500 4650 50  0001 C CNN
+F 0 "#PWR031" H 7500 4650 50  0001 C CNN
 F 1 "GND" H 7500 4750 50  0000 C CNN
 F 2 "" H 7500 4900 50  0000 C CNN
@@
 	7500 4500 7700 4500
 $Comp
-L C C?
+L C C7
 U 1 1 58987CEA
 P 9450 5800
-F 0 "C?" H 9475 5900 50  0000 L CNN
+F 0 "C7" H 9475 5900 50  0000 L CNN
 F 1 "4.7uf" H 9475 5700 50  0000 L CNN
 F 2 "Capacitors_SMD:C_0603" H 9488 5650 50  0001 C CNN
