File: esp32bb.sch (KiCad schematic (older format))
At the start: 31 parts, among them CON1 Micro_SD_Card, IC1 FT232RQ, P1 CONN_01X17, P2 CONN_01X17, P3 USB_OTG, Q1 MMBT3904, Q2 MMBT3904, SW1 SWITCH_SPST, SW2 SWITCH_SPST, U1 ESP32-WROOM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

Commit message: Rename project name to esp32bb
Parts:
- P3: symbol USB_OTG-RESCUE-esp-wroom-32-break -> USB_OTG-RESCUE-esp32bb
Changed lines of the file:
@@
 EESchema Schematic File Version 2
-LIBS:esp-wroom-32-break-rescue
+LIBS:esp32bb-rescue
 LIBS:power
 LIBS:device
@@
 LIBS:ftdi232rq
 LIBS:MiscellaneousDevices
-LIBS:esp-wroom-32-break-cache
+LIBS:esp32bb-cache
 EELAYER 25 0
 EELAYER END
@@
 $EndComp
 $Comp
-L USB_OTG-RESCUE-esp-wroom-32-break P3
+L USB_OTG-RESCUE-esp32bb P3
 U 1 1 586B58B7
 P 10650 4150
