File: main_pcb/esp32bb.sch (KiCad schematic (older format))
At the start: 27 parts, among them P1 CONN_01X17, P2 CONN_01X17, P3 USB_OTG, Q1 MMBT3904, Q2 MMBT3904, SW1 SWITCH_SPST, SW2 SWITCH_SPST, U1 ESP32-WROOM, U2 NCP1117ST33T3G, U3 CP2102

Commit message: Create main_pcb directory
Parts:
- added Q?: Q_NMOS_DGS, symbol Device:Q_NMOS_DGS
- C1, C2, C3, C4, C5, C6, C7, C8: symbol C -> esp32bb-rescue:C
- D1, D2: footprint Diodes_SMD:D_0805 -> common:D_0805; symbol D -> esp32bb-rescue:D
- D3: symbol LED -> esp32bb-rescue:LED
- P1, P2: symbol CONN_01X17 -> esp32bb-rescue:CONN_01X17
- P3: symbol USB_OTG-RESCUE-esp32bb -> esp32bb-rescue:USB_OTG-RESCUE-esp32bb
- Q1, Q2: symbol MMBT3904 -> esp32bb-rescue:MMBT3904
- R1, R2, R3, R4, R5, R6: symbol R -> esp32bb-rescue:R
- SW1, SW2: symbol SWITCH_SPST -> esp32bb-rescue:SWITCH_SPST
- U1: symbol ESP32-WROOM -> esp32bb-rescue:ESP32-WROOM
- U2: symbol NCP1117ST33T3G -> esp32bb-rescue:NCP1117ST33T3G
- U3: symbol CP2102 -> esp32bb-rescue:CP2102
Connections:
- wire segments 77 -> 96
